File: analogboard/pcb/SOL_AMPV2.brd (EAGLE design)
At the start: 65.2 x 118.6 mm, 308 parts, among them IC1 LM1117, IC2 LM1117, T1 UA_TPPAD1-13, T10 UA_TPPAD1-13, T11 UA_TPPAD1-13, T13 UA_TPPAD1-13, T14 UA_TPPAD1-13, T15 UA_TPPAD1-13, T16 UA_TPPAD1-13, T17 UA_TPPAD1-13, T2 UA_TPPAD1-13, T3 UA_TPPAD1-13, T4 UA_TPPAD1-13, T5 UA_TPPAD1-13, T9 UA_TPPAD1-13, U1 MCP4728-E/UN, U2 MCP4728-E/UN, U3 ADL5317, U4 MCP4725A0T-E/CH, U5 MCP9808-E/MS, U8 P82B715TD, X1 40pin, X2 22-23-2021, X3 22-23-2021, X4 22-23-2041, X5 DIN41612_ABC_96_R

Commit message: files sent for production
Parts:
- added LDAC1, LDAC2: UA_TPPAD1-13, UA_v2:UA_P1-13
- R11, R5: value 0E -> 4.7K; device resistor:R0402 -> UA_v2:R0805H
- moved R5 2.86 mm to (7.94, 113.0), turned to 0 degrees
- moved R11 1.00 mm to (6.35, 30.5), turned to 0 degrees
- moved R12 0.32 mm to (3.81, 28.3)
Connections:
- removed net N$12: R11.2, R12.1, U2.4
- removed net N$8: R5.2, R6.1, U1.4
- new net LDAC1: LDAC1.TP, R5.2, R6.1, U1.4
- new net LDAC2: LDAC2.TP, R11.2, R12.1, U2.4
Routing:
- net LDAC2: track 0.00 -> 9.06 mm
- net LDAC1: track 0.00 -> 8.32 mm
- net N$12: track 6.63 -> 0.00 mm
- net N$8: track 6.45 -> 0.00 mm
- net GND: track 115.5 -> 110.7 mm
- net N$11: track 19.2 -> 18.1 mm
Other:
- board text added: "SOLID Amplifier V2.0.1 20150921 W.Beaumont"
- board text added: "SOLID Amplifier V2.0.1 20150921 W.Beaumont Universiteit Antwerpen"
- board text removed: "SOLID Amplifier V2.0 20150918 W.Beaumont"
- board text removed: "SOLID Amplifier V2.0 20150918 W.Beaumont Universiteit Antwerpen"
