File: analogboard/pcb/SOL_AMPV2.sch (EAGLE design)
At the start: 71 parts, among them IC1 LM1117, IC2 LM1117, T1 UA_TPPAD1-13, T10 UA_TPPAD1-13, T11 UA_TPPAD1-13, T13 UA_TPPAD1-13, T14 UA_TPPAD1-13, T15 UA_TPPAD1-13, T16 UA_TPPAD1-13, T17 UA_TPPAD1-13, T2 UA_TPPAD1-13, T3 UA_TPPAD1-13, T4 UA_TPPAD1-13, T5 UA_TPPAD1-13, T9 UA_TPPAD1-13, U1 MCP4728-E/UN, U2 MCP4728-E/UN, U3 ADL5317, U4 MCP4725A0T-E/CH, U5 MCP9808-E/MS, U8 P82B715TD, X1 40pin, X2 22-23-2021, X3 22-23-2021, X4 22-23-2041, X5 DIN41612_ABC_96_R

Commit message: files sent for production
Parts:
- added LDAC1, LDAC2: UA_TPPAD1-13, UA_v2:UA_TPPAD1-13
- R11, R5: value 0E -> 4.7K; device resistor:R-EU_R0402 -> UA_v2:R_HAND
Connections:
- removed net N$12: R11.2, R12.1, U2.*LDAC
- removed net N$8: R5.2, R6.1, U1.*LDAC
- new net LDAC1: LDAC1.TP, R5.2, R6.1, U1.*LDAC
- new net LDAC2: LDAC2.TP, R11.2, R12.1, U2.*LDAC
Other:
- moved on the sheet: C2, R10, R12, U1, U2
