File: sensorboard/board/panel13_13.kicad_pcb (KiCad board)
At the start: 2 copper layers, 181 x 426 mm, 169 parts, among them U11101 SiPM_Socket, U111010 SiPM_Socket, U111011 SiPM_Socket, U111012 SiPM_Socket, U111013 SiPM_Socket, U11102 SiPM_Socket, U11103 SiPM_Socket, U11104 SiPM_Socket, U11105 SiPM_Socket, U11106 SiPM_Socket, U11107 SiPM_Socket, U11108 SiPM_Socket, U11109 SiPM_Socket, U1111 SiPM_Socket, U11110 SiPM_Socket, U11111 SiPM_Socket, U111110 SiPM_Socket, U111111 SiPM_Socket, U111112 SiPM_Socket, U111113 SiPM_Socket, U11112 SiPM_Socket, U11113 SiPM_Socket, U11114 SiPM_Socket, U11115 SiPM_Socket, U11116 SiPM_Socket, U11117 SiPM_Socket, U11118 SiPM_Socket, U11119 SiPM_Socket, U1112 SiPM_Socket, U11121 SiPM_Socket, U111210 SiPM_Socket, U111211 SiPM_Socket, U111212 SiPM_Socket, U111213 SiPM_Socket, U11122 SiPM_Socket, U11123 SiPM_Socket, U11124 SiPM_Socket, U11125 SiPM_Socket, U11126 SiPM_Socket, U11127 SiPM_Socket, U11128 SiPM_Socket, U11129 SiPM_Socket, U1113 SiPM_Socket, U11131 SiPM_Socket, U111310 SiPM_Socket, U111311 SiPM_Socket, U111312 SiPM_Socket, U111313 SiPM_Socket, U11132 SiPM_Socket, U11133 SiPM_Socket, U11134 SiPM_Socket, U11135 SiPM_Socket, U11136 SiPM_Socket, U11137 SiPM_Socket, U11138 SiPM_Socket, U11139 SiPM_Socket, U1114 SiPM_Socket, U1115 SiPM_Socket, U1116 SiPM_Socket, U1117 SiPM_Socket, U1118 SiPM_Socket, U1119 SiPM_Socket, U1121 SiPM_Socket, U11210 SiPM_Socket, U11211 SiPM_Socket, U11212 SiPM_Socket, U11213 SiPM_Socket, U1122 SiPM_Socket, U1123 SiPM_Socket, U1124 SiPM_Socket, U1125 SiPM_Socket, U1126 SiPM_Socket, U1127 SiPM_Socket, U1128 SiPM_Socket, U1129 SiPM_Socket, U1131 SiPM_Socket, U11310 SiPM_Socket, U11311 SiPM_Socket, U11312 SiPM_Socket, U11313 SiPM_Socket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

Commit message: Cleaning up repo for old 13x7 panel.
Parts:
- added FID0: Fiducial_Modern_CopperTop, Fiducials:Fiducial_Modern_CopperTop, F.Cu at (12.0, 22.0)
- added FID1: Fiducial_Modern_CopperTop, Fiducials:Fiducial_Modern_CopperTop, F.Cu at (188.0, 22.0)
- added FID2: Fiducial_Modern_CopperTop, Fiducials:Fiducial_Modern_CopperTop, F.Cu at (12.0, 425.0)
- added FID3: Fiducial_Modern_CopperTop, Fiducials:Fiducial_Modern_CopperTop, F.Cu at (188.0, 425.0)
Other:
- board size 181 x 426 mm -> 190 x 426 mm
- board text added: "SiPM orientation"
Changed lines of the file:
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@@
 (kicad_pcb (version 4) (host pcbnew 4.0.2-4+6225~38~ubuntu14.04.1-stable)
   (general
-    (links 3)
-    (no_connects 0)
-    (area 9.949999 10.949999 191.050001 437.275782)
+    (links 0)
+    (no_connects 504)
+    (area 2.273354 10.949999 199.347166 437.275782)
     (thickness 1.6)
-    (drawings 13799)
+    (drawings 13814)
     (tracks 3380)
     (zones 0)
-    (modules 169)
+    (modules 173)
     (nets 4)
   )
-  (page User 229.997 489.991)
+  (page A3 portrait)
   (title_block
     (title "SiPM to IDC4")
@@
   )
   (layers
-    (0 F.Cu signal hide)
-    (31 B.Cu signal hide)
+    (0 F.Cu signal)
+    (31 B.Cu signal)
     (32 B.Adhes user)
     (33 F.Adhes user)
@@
     (pcbplotparams
       (layerselection 0x010fc_80000001)
-      (usegerberextensions true)
+      (usegerberextensions false)
       (excludeedgelayer true)
       (linewidth 0.100000)
@@
     (add_net "Net-(U1-Pad4)")
   )
+  (module Fiducials:Fiducial_Modern_CopperTop (layer F.Cu)
+    (at 12 22)
+    (descr "Fiducial, Modern, Copper Top, Passermarke,")
+    (tags "Fiducial, Modern, Copper Top, Passermarke,")
+    (fp_text reference FID0 (at -2.75 8.25) (layer F.SilkS)
+      (effects (font (size 1 1) (thickness 0.15)))
+    )
+    (fp_text value Fiducial_Modern_CopperTop (at 0.81026 4.18084) (layer F.Fab)
+      (effects (font (size 1 1) (thickness 0.15)))
+    )
+    (fp_circle (center 0 0) (end 1.52908 0) (layer F.Cu) (width 0.381))
+    (fp_circle (center 0 0) (end 1.7907 0) (layer F.Cu) (width 0.381))
+    (pad ~ smd circle (at 0 0) (size 4.8006 4.8006) (layers F.Mask)
+      (solder_mask_margin 2.99974))
+  )
+  (module Fiducials:Fiducial_Modern_CopperTop (layer F.Cu)
+    (at 188 425)
+    (descr "Fiducial, Modern, Copper Top, Passermarke,")
+    (tags "Fiducial, Modern, Copper Top, Passermarke,")
+    (fp_text reference FID3 (at 1 -8.25) (layer F.SilkS)
+      (effects (font (size 1 1) (thickness 0.15)))
+    )
+    (fp_text value Fiducial_Modern_CopperTop (at 0.81026 4.18084) (layer F.Fab)
+      (effects (font (size 1 1) (thickness 0.15)))
+    )
+    (fp_circle (center 0 0) (end 1.52908 0) (layer F.Cu) (width 0.381))
+    (fp_circle (center 0 0) (end 1.7907 0) (layer F.Cu) (width 0.381))
+    (pad ~ smd circle (at 0 0) (size 4.8006 4.8006) (layers F.Mask)
+      (solder_mask_margin 2.99974))
+  )
+  (module Fiducials:Fiducial_Modern_CopperTop (layer F.Cu)
+    (at 188 22)
+    (descr "Fiducial, Modern, Copper Top, Passermarke,")
+    (tags "Fiducial, Modern, Copper Top, Passermarke,")
+    (fp_text reference FID1 (at 1 9) (layer F.SilkS)
+      (effects (font (size 1 1) (thickness 0.15)))
+    )
+    (fp_text value Fiducial_Modern_CopperTop (at 0.81026 4.18084) (layer F.Fab)
+      (effects (font (size 1 1) (thickness 0.15)))
+    )
+    (fp_circle (center 0 0) (end 1.52908 0) (layer F.Cu) (width 0.381))
+    (fp_circle (center 0 0) (end 1.7907 0) (layer F.Cu) (width 0.381))
+    (pad ~ smd circle (at 0 0) (size 4.8006 4.8006) (layers F.Mask)
+      (solder_mask_margin 2.99974))
+  )
   (module sipm_socket:sipm_socket (layer F.Cu)
     (at 169 429.5)
@@
       (net 2 "Net-(U1-Pad3)"))
   )
-  (gr_line (start 186.75 230.25) (end 186.75 250.25) (layer F.SilkS) (width 5))
-  (gr_text "Hamamatsu Box #" (at 187 205.25 270) (layer F.SilkS)
+  (module Fiducials:Fiducial_Modern_CopperTop (layer F.Cu)
+    (at 12 425)
+    (descr "Fiducial, Modern, Copper Top, Passermarke,")
+    (tags "Fiducial, Modern, Copper Top, Passermarke,")
+    (fp_text reference FID2 (at -1.25 -7.75) (layer F.SilkS)
+      (effects (font (size 1 1) (thickness 0.15)))
+    )
+    (fp_text value Fiducial_Modern_CopperTop (at 0.81026 4.18084) (layer F.Fab)
+      (effects (font (size 1 1) (thickness 0.15)))
+    )
+    (fp_circle (center 0 0) (end 1.52908 0) (layer F.Cu) (width 0.381))
+    (fp_circle (center 0 0) (end 1.7907 0) (layer F.Cu) (width 0.381))
+    (pad ~ smd circle (at 0 0) (size 4.8006 4.8006) (layers F.Mask)
+      (solder_mask_margin 2.99974))
+  )
+  (gr_text "SiPM\norientation" (at 187.5 60.5) (layer F.SilkS)
+    (effects (font (size 1.5 1.5) (thickness 0.3)))
+  )
+  (gr_line (start 188.75 55) (end 188.5 55) (layer F.SilkS) (width 0.2))
+  (gr_line (start 188.75 56.25) (end 188.75 55) (layer F.SilkS) (width 0.2))
+  (gr_line (start 188.5 56.25) (end 188.75 56.25) (layer F.SilkS) (width 0.2))
+  (gr_line (start 188.5 55) (end 188.5 56.25) (layer F.SilkS) (width 0.2))
+  (gr_line (start 185.5 56) (end 185.5 55) (layer F.SilkS) (width 0.2))
+  (gr_line (start 185.25 56.25) (end 185.5 56) (layer F.SilkS) (width 0.2))
+  (gr_line (start 185.25 55) (end 185.25 56.25) (layer F.SilkS) (width 0.2))
+  (gr_line (start 192.5 56.25) (end 192.5 55) (layer F.SilkS) (width 0.2))
+  (gr_line (start 182.5 56.25) (end 192.5 56.25) (layer F.SilkS) (width 0.2))
+  (gr_line (start 182.5 55) (end 182.5 56.25) (layer F.SilkS) (width 0.2))
+  (gr_line (start 192.5 45) (end 182.5 45) (layer F.SilkS) (width 0.2))
+  (gr_line (start 192.5 55) (end 192.5 45) (layer F.SilkS) (width 0.2))
+  (gr_line (start 182.5 55) (end 192.5 55) (layer F.SilkS) (width 0.2))
+  (gr_line (start 182.5 45) (end 182.5 55) (layer F.SilkS) (width 0.2))
+  (gr_line (start 189.25 230.25) (end 189.25 250.25) (layer F.SilkS) (width 5))
+  (gr_text "Hamamatsu Box #" (at 189.25 205.25 270) (layer F.SilkS)
     (effects (font (size 3 3) (thickness 0.3)))
   )
@@
     (effects (font (size 3 3) (thickness 0.3)))
   )
-  (gr_line (start 10 437) (end 10 11) (layer Edge.Cuts) (width 0.1))
-  (gr_line (start 10 437) (end 191 437) (layer Edge.Cuts) (width 0.1))
-  (gr_line (start 191 11) (end 191 437) (layer Edge.Cuts) (width 0.1))
-  (gr_line (start 10 11) (end 191 11) (layer Edge.Cuts) (width 0.1))
+  (gr_line (start 5 437) (end 5 11) (layer Edge.Cuts) (width 0.1))
+  (gr_line (start 5 437) (end 195 437) (layer Edge.Cuts) (width 0.1))
+  (gr_line (start 195 11) (end 195 437) (layer Edge.Cuts) (width 0.1))
+  (gr_line (start 5 11) (end 195 11) (layer Edge.Cuts) (width 0.1))
   (gr_line (start 172 424) (end 173 424) (layer B.SilkS) (width 5))
   (gr_line (start 159.5 424) (end 160.5 424) (layer B.SilkS) (width 5))
